Commit message: Moving laser scanner in front for gazebo

File: gazebo/gazebo_robile.xacro (robot description, xacro)
@@ -48,5 +48,5 @@
     <!-- base laser front -->
     <xacro:hokuyo_urg04_laser name="base_laser_front" parent="base" ros_topic="scan" update_rate="10" min_angle="-3.14" max_angle="3.14">
-    <origin xyz="0.0 0.0 0.3" rpy="0.0 0.0 0.0"/>
+    <origin xyz="0.466 0.0 0.2" rpy="0.0 0.0 0.0"/>
     </xacro:hokuyo_urg04_laser>
 </robot>

File: gazebo/gazebo_ros_planar_move.xacro (robot description, xacro)
@@ -48,6 +48,7 @@
             <publish_odom_tf>true</publish_odom_tf>
             <!-- Frame IDs -->
-            <odometry_frame>odom</odometry_frame>
-            <robot_base_frame>base_link</robot_base_frame>
+            <!-- For multi robot these values get modified in generic_spawn.py -->
+	    <odometry_frame>odom</odometry_frame>
+	    <robot_base_frame>base_link</robot_base_frame>
             <!-- Set odom covariance -->
             <covariance_x>0.0001</covariance_x>
